Commit message: Ready for commit
- Add customized world
- Correct robot's camera frame
- Change launch files and script

File: urdf/my_bot.xacro (robot description, xacro)
@@ -137,5 +137,5 @@
   </joint>
   <!-- camera -->
-  <link name='camera'>
+  <link name='camera_link'>
     <inertial>
       <mass value="0.1"/>
@@ -162,5 +162,5 @@
   <joint type="fixed" name="camera_joint">
     <origin xyz="0.1 0 0" rpy="0 0 0"/>
-    <child link="camera"/>
+    <child link="camera_link"/>
     <parent link="chassis"/>
   </joint>
@@ -169,5 +169,5 @@
     <origin xyz="0 0 0" rpy="0 0 0"/>
     <child link="camera_rgbd_frame"/>
-    <parent link="camera"/>
+    <parent link="camera_link"/>
   </joint>
   <!-- hokuyo laser rangefinder -->
@@ -191,5 +191,5 @@
       <origin xyz="0.0 0 0" rpy=" 0 0 0"/>
       <geometry>
-        <mesh filename="package://my_bot/meshes/hokuyo.dae"/>
+        <mesh filename="package://slam_project/meshes/hokuyo.dae"/>
       </geometry>
     </visual>
